Commit message: v24.10.19_18:27 Update joint_names in RobotSimNode constructor

File: ros2_ws/src/rrm/rrm_simple_robot_model/urdf/arm.urdf (robot description, URDF)
Before this commit: robot arm, 8 links, 7 joints
Links:
- added link link_4_5; visual sphere radius=0.03
- added link link_5; visual cylinder length=0.15 radius=0.01
Joints:
- added joint joint_4_5: type fixed, parent link_4, child link_4_5, origin xyz=0 0 0.05 rpy=0 0 0
- added joint joint_5: type revolute, parent link_4_5, child link_5, origin xyz=0 0 0 rpy=0 0 0, axis 0 1 0, limit lower=-0.96 upper=2.182 effort=1000.0 velocity=0.5
- joint joint_tool0: origin xyz=0 0 0.05 rpy=0 0 0 -> xyz=0 0 0.15 rpy=0 0 0; parent link_4 -> link_5
