Commit message: v24.10.19_18:20 Update robot_sim_node.cpp to include joint_4 in joint_names

File: ros2_ws/install/rrm_simple_robot_model/share/rrm_simple_robot_model/urdf/arm.urdf (robot description, URDF)
Before this commit: robot arm, 6 links, 5 joints
Links:
- added link link_3_4; visual sphere radius=0.03
- added link link_4; visual cylinder length=0.05 radius=0.01
- link tool0: geometry visual sphere radius=0.03
Joints:
- removed joint joint_3-tool0
- added joint joint_3_4: type fixed, parent link_3, child link_3_4, origin xyz=0 0 0.203 rpy=0 0 0
- added joint joint_4: type revolute, parent link_3, child link_4, origin xyz=0 0 0.203 rpy=0 0 0, axis 0 1 0, limit lower=-0.96 upper=2.182 effort=1000.0 velocity=0.5
- added joint joint_tool0: type fixed, parent link_4, child tool0, origin xyz=0 0 0.05 rpy=0 0 0

Commit message: v24.10.19_18:43 Refactor build and URDF files

File: ros2_ws/install/rrm_simple_robot_model/share/rrm_simple_robot_model/urdf/arm.urdf (robot description, URDF)
Before this commit: robot arm, 10 links, 9 joints
Links:
- link tool0: geometry 

Commit message: v24.10.23_15:53 Update stderr.log files

File: ros2_ws/install/rrm_simple_robot_model/share/rrm_simple_robot_model/urdf/arm.urdf (robot description, URDF)
Before this commit: robot arm, 10 links, 9 joints
Links:
- link link_1: geometry visual sphere radius=0.01
- link link_2: geometry visual cylinder length=0.203 radius=0.01
Joints:
- joint joint_1: origin xyz=0 0 0 rpy=0 0 0 -> xyz=0 0 0.005 rpy=0 0 0
- joint joint_2: origin xyz=0 0 0 rpy=0 0 0 -> xyz=0 0 0.01 rpy=0 0 0
- joint joint_5: origin xyz=0 0 0 rpy=0 0 0 -> xyz=0 0 0.03 rpy=0 0 0

Commit message: v24.10.23_16:30 Add empty stderr.log files for build logs

File: ros2_ws/install/rrm_simple_robot_model/share/rrm_simple_robot_model/urdf/arm.urdf (robot description, URDF)
Before this commit: robot arm, 10 links, 9 joints
Links:
- added link link_5_6; visual sphere radius=0.03
- added link link_6; visual cylinder length=0.0 radius=0.01
- link link_1: geometry visual sphere radius=0.0
Joints:
- added joint joint_5_6: type fixed, parent link_5, child link_5_6, origin xyz=0 0 0.15 rpy=0 0 0
- added joint joint_6: type prismatic, parent link_5_6, child link_6, origin xyz=0 0 0.03 rpy=0 0 0, axis 0 0 1, limit lower=0.0 upper=0.1 effort=1000.0 velocity=0.5
- joint joint_3: origin xyz=0 0 0.203 rpy=0 0 0 -> xyz=0 0 0.03 rpy=0 0 0; parent link_2 -> link_2_3
- joint joint_4: axis 0 1 0 -> 0 0 1; limit lower=-0.96 upper=2.182 effort=1000.0 velocity=0.5 -> lower=-3.14 upper=3.14 effort=1000.0 velocity=0.5; origin xyz=0 0 0.203 rpy=0 0 0 -> xyz=0 0 0.03 rpy=0 0 0; parent link_3 -> link_3_4
- joint joint_5: limit lower=-0.96 upper=2.182 effort=1000.0 velocity=0.5 -> lower=-2.2 upper=2.2 effort=1000.0 velocity=0.5
- joint joint_tool0: origin xyz=0 0 0.15 rpy=0 0 0 -> xyz=0 0 0 rpy=0 0 0; parent link_5 -> link_6

Commit message: v24.11:13_21:38 add empty log files for Zad1.6 and stderr outputs

File: ros2_ws/install/rrm_simple_robot_model/share/rrm_simple_robot_model/urdf/arm.urdf (robot description, URDF)
Before this commit: robot arm, 12 links, 11 joints
Links:
- link link_6: geometry visual cylinder length=0 radius=0.01
